File: Hardware/Basic/Top/WatchMe-BASIC-TOP.brd (EAGLE design)
At the start: 38 x 38 mm, 29 parts, among them U2 NRF52832_MODULE_MDBT42

Commit message: updated top brd/sch
Parts:
- added C2, C5, C6: 1u, LinnesLab-Passives:C0603
- added C20, C21: 4.7u, LinnesLab-Passives:C0603
- added CHRG2: MCP73831, LinnesLab-Power:SOT23-5
- added D4, D5: (no value), LinnesLab-DiscreteSemi:USC
- added J2: (no value), LinnesLab-Connectors:1X02
- added LDO2: MIC5504, LinnesLab-Power:SOT23-5
- added R11: (no value), LinnesLab-Passives:R0603
- added R12, R13, R14, R15: 100k, LinnesLab-Passives:R0603
- added R8, R9: 10k, LinnesLab-Passives:R0603
- added SW1, SW2: SWITCH.MOM, LinnesLab-Switches:TACTILE_SWITCH_SMD_6.2MM_TALL
- added U4: PCF8523, LinnesLab-Clocks:SO8
- added USB2: USB.MICRO-BIGGERPADS, LinnesLab-Connectors:USB-MICRO-01.BIGGERPADS
- added XTAL3: 32.7680kHz, LinnesLab-Clocks:2-SMD.NOLEAD.2.0MMTO1.2MM
Connections:
- new net BATT: R13.1, R14.2
- new net CHRG.STAT: CHRG2.1, R12.1
- new net N$17: CHRG2.5, R11.2
- new net N$19: U4.2, XTAL3.P$1
- new net N$20: U4.1, XTAL3.P$2
- new net SW1: SW1.A1, SW2.A1
- new net USB+: USB2.3
- new net USB-: USB2.2
- new net VBATT: U4.3
- new net VIN: C21.2, C5.2, CHRG2.4, D4.-, D5.-, LDO2.1, LDO2.3, R12.2
- new net VLIPO: C20.1, CHRG2.3, D4.+, J2.2, R13.2
- new net V_USB: D5.+, USB2.1
- net 3.3V: now also C2.1, C6.1, LDO2.5, R15.2, R8.2, R9.2, U4.8
- net GND: now also C2.2, C20.2, C21.1, C5.1, C6.2, CHRG2.2, J2.1, LDO2.2, R11.1, R14.1, R15.1, SW1.B1, SW1.B2, SW2.B1, SW2.B2, U4.4, USB2.5
- net SCL: now also R8.1, U4.6
- net SDA: now also R9.1, U4.5

Commit message: updated top board/sch
Parts:
- added C22: 100n, LinnesLab-Passives:C0603
- added C23, C24: 47p, LinnesLab-Passives:C0603
- added J3: (no value), LinnesLab-Connectors:1X06_1.27MM
- added JP2: (no value), LinnesLab-Switches:SMT-JUMPER_2_NO_SILK
- added LED5: RED, LinnesLab-LED:LED-0603
- added LED6: YELLOW, LinnesLab-LED:LED-0603
- added R1, R2: 10k, LinnesLab-Passives:R0603
- added R17, R18: 27, LinnesLab-Passives:R0603
- added R19, R20: 1k, LinnesLab-Passives:R0603
- added U5: FT231XS, LinnesLab-DigitalIC:SSOP20_L
- R8, R9: value 10k -> 0
- moved R9 49.4 mm to (-20.5, -12.3), turned to 0 degrees
- moved R8 46.7 mm to (-20.5, -9.65), turned to 0 degrees
Connections:
- removed net BATT: R13.1, R14.2
- removed net CD1: SD2.CD1
- removed net CHRG.STAT: CHRG2.1, R12.1
- removed net CS.OLED: U3.13
- removed net DC.OLED: U3.15
- removed net RESET.OLED: U3.14
- removed net RXD: U2.21
- removed net SD.CS: SD2.2
- removed net SW1: SW1.A1, SW2.A1
- removed net TXD: U2.19
- new net !CTS: JP2.2, U5.9
- new net !DTR: U5.1
- new net A4/BATT: R13.1, R14.2, U2.5
- new net A6/TIA: U2.7
- new net A7/PPG: U2.8
- new net D11/SW1: SW1.A1, U2.25
- new net D15/SW2: SW2.A1, U2.29
- new net D16/CS.OLED: U2.30, U3.13
- new net D27/CHRG.STATUS: CHRG2.1, R12.1, U2.4
- new net D29/LED.CTRL: U2.6
- new net D3/RESET.OLED: U2.16, U3.14
- new net D4/DC.OLED: U2.17, U3.15
- new net D5/CD1: SD2.CD1, U2.18
- new net D7/SD.CS: SD2.2, U2.20
- new net FT3V3: U5.13
- new net N$23: R17.2, U5.12
- new net N$24: R18.2, U5.11
- new net N$25: LED5.C, R19.2
- new net N$26: LED6.C, R20.2
- new net RXD.FT: R9.1, U5.4
- new net RXD.NRF: R8.2, U2.21
- new net RXLED: R19.1, U5.17
- new net TXD.FT: R8.1, U5.20
- new net TXD.NRF: R9.2, U2.19
- new net TXLED: R20.1, U5.10
- net 3.3V: now also C22.2, LED5.A, LED6.A, R1.2, R2.2, U5.14, U5.3; no longer R8.2, R9.2
- net GND: now also C22.1, C23.2, C24.1, JP2.1, U5.16, U5.6
- net SCL: now also R2.1; no longer R8.1
- net SDA: now also R1.1; no longer R9.1
- net USB+: now also C23.1, R18.1
- net USB-: now also C24.2, R17.1
- net V_USB: now also U5.15
