File: Hardware/Basic/Top/WatchMe-BASIC-TOP_withtempsensor.brd (EAGLE design)
At the start: 38 x 38 mm, 65 parts, among them SW1 SWITCH.MOM, SW2 SWITCH.MOM, U2 NRF52832_MODULE_MDBT42, U4 PCF8523, U5 FT231XS

Commit message: updated top board/sch again
Parts:
- added C3: 100n, LinnesLab-Passives:C0603
- added R22, R23, R24: 10k, LinnesLab-Passives:R0603
- added U6: MCP9808-MSOP8, LinnesLab-Sensors:MSOP08
- moved R9 49.9 mm to (-20.5, -12.3), turned to 0 degrees
- moved R8 45.3 mm to (-20.5, -9.65), turned to 0 degrees
- moved C2 40.2 mm to (7.95, 28.0)
- moved R20 33.5 mm to (-3.20, 26.3), turned to 0 degrees
- moved LED6 29.5 mm to (-3.20, 33.9), turned to 0 degrees
- moved R19 26.3 mm to (-3.20, 30.1)
- moved XTAL3 22.7 mm to (1.57, 25.9)
- moved U4 22.3 mm to (6.15, 24.4)
- moved R2 21.6 mm to (-20.5, -5.56)
- moved LED5 21.5 mm to (-3.20, 37.7), turned to 0 degrees
- moved LDO2 19.4 mm to (8.13, 6.35)
- moved JP2 18.4 mm to (-20.7, 29.2)
- moved U5 18.3 mm to (-14.0, 32.6)
- moved R1 18.3 mm to (-20.5, -2.87)
- moved C5 18.1 mm to (4.65, 6.22), turned to 90 degrees
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Connections:
- new net ALERT: R24.1
- new net D2/DT.ALERT: U2.15, U6.3
- net 3.3V: now also C3.1, R22.2, R23.2, R24.2, U6.8
- net GND: now also C3.2, U6.4, U6.5, U6.6, U6.7
- net SCL: now also R23.1, U6.2
- net SDA: now also R22.1, U6.1
