File: Hardware/Basic/Top/WatchMe-BASIC-TOP_withtempsensor.sch (EAGLE design)
At the start: 65 parts, among them SW1 SWITCH.MOM, SW2 SWITCH.MOM, U2 NRF52832_MODULE_MDBT42, U4 PCF8523, U5 FT231XS

Commit message: updated top board/sch again
Parts:
- added C3: 100n, LinnesLab-Passives:CAPACITOR0603
- added R22, R23, R24: 10k, LinnesLab-Passives:RESISTOR0603
- added U6: MCP9808-MSOP8, LinnesLab-Sensors:MCP9808-MSOP8
Connections:
- new net ALERT: R24.1
- new net D2/DT.ALERT: U2.P0.02/AIN0, U6.ALERT
- net 3.3V: now also C3.1, R22.2, R23.2, R24.2, U6.VDD
- net GND: now also C3.2, U6.A0, U6.A1, U6.A2, U6.GND
- net SCL: now also R23.1, U6.SCL
- net SDA: now also R22.1, U6.SDA
Other:
- note added: "I2C Adress: A0,A1,A2 connected to ground: 0x18 Other addresses: 0x19 to 0x1F"
- note added: "MCP9808 Digital Temperature Sensor"
- moved on the sheet: CORTEX1
